File: v5/kicad/binary_clock.kicad_pcb (KiCad board)
At the start: 2 copper layers, 18 parts, among them J1 AVR-ISP-6, SW1 SW_Push, SW2 SW_Push, SW3 SW_Push, U1 ATmega48A-P, Y1 Crystal

Commit message: Add files via upload
Parts:
- BT1: footprint Battery:BatteryHolder_Keystone_104_1x23mm -> Battery:BatteryHolder_Keystone_103_1x20mm
- D1, D10, D11, D2, D3, D4, D5, D6, D7, D8, D9: footprint LED_SMD:LED_1210_3225Metric_Pad1.42x2.65mm_HandSolder -> LED_THT:LED_D3.0mm
- J1: footprint Connector_PinHeader_2.00mm:PinHeader_2x03_P2.00mm_Vertical -> Connector_PinSocket_2.54mm:PinSocket_2x03_P2.54mm_Vertical
- SW1, SW2, SW3: footprint Button_Switch_SMD:SW_Push_1P1T_NO_CK_KSC6xxJ -> Button_Switch_THT:SW_PUSH_6mm
- Y1: footprint Crystal:Crystal_AT310_D3.0mm_L10.0mm_Vertical -> Crystal:Crystal_DS10_D1.0mm_L4.3mm_Vertical
- moved D6 47.0 mm to (124.1, 60.1)
- moved D7 39.1 mm to (118.1, 67.1), turned to -90 degrees
- moved J1 36.0 mm to (40.5, 63.0), turned to -90 degrees
- moved BT1 33.9 mm to (89.8, 42.0)
- moved SW1 33.5 mm to (53.1, 78.5), turned to -90 degrees
- moved SW2 30.3 mm to (58.4, 85.0), turned to 90 degrees
- moved D8 29.9 mm to (112.1, 67.1), turned to -90 degrees
- moved U1 25.0 mm to (48.2, 67.7), turned to 90 degrees
- moved SW3 25.0 mm to (68.6, 85.0), turned to 90 degrees
- moved D10 23.6 mm to (100.1, 67.1), turned to -90 degrees
- moved D11 23.6 mm to (94.1, 67.1), turned to -90 degrees
- moved D9 23.3 mm to (106.1, 67.1), turned to -90 degrees
- moved Y1 14.9 mm to (70.6, 71.8), turned to 180 degrees
- moved D1 14.7 mm to (94.1, 60.1)
- moved D2 14.7 mm to (100.1, 60.1)
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Connections:
- D10 pad 1: Net-(D1-K) -> Net-(D10-K)
- D11 pad 1: Net-(D1-K) -> Net-(D10-K)
- D7 pad 1: Net-(D1-K) -> Net-(D10-K)
- D8 pad 1: Net-(D1-K) -> Net-(D10-K)
- D9 pad 1: Net-(D1-K) -> Net-(D10-K)
- U1 pad 16: unconnected-(U1-PB2-Pad16) -> Net-(D10-K)
- U1 pad 20: +3.3V -> unconnected-(U1-AVCC-Pad20)
- U1 pad 21: +3.3V -> unconnected-(U1-AREF-Pad21)
Routing:
- net Net-(D1-K): track 120.6 -> 43.0 mm
- net Net-(D6-A): track 11.0 -> 84.9 mm
- net Net-(D8-A): track 0.00 -> 66.7 mm
- net MOSI: track 0.00 -> 57.9 mm, vias 0 -> 2
- net Net-(D7-A): track 27.1 -> 76.2 mm
- net +3.3V: track 46.9 -> 90.5 mm, vias 0 -> 2
- net Net-(D10-K): track 0.00 -> 43.0 mm
- net Net-(D5-A): track 38.1 -> 75.2 mm
- net Net-(D9-A): track 0.00 -> 36.7 mm
- net Net-(D4-A): track 31.0 -> 65.5 mm
- net SCK: track 10.0 -> 42.3 mm
- net Net-(D3-A): track 24.0 -> 55.8 mm
- net Net-(D2-A): track 16.9 -> 46.1 mm
- net Net-(D10-A): track 0.00 -> 27.0 mm
- net Net-(D1-A): track 9.89 -> 36.4 mm
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
Commit message: Add files via upload
Parts:
- added R1: 4.7k, Resistor_THT:R_Axial_DIN0207_L6.3mm_D2.5mm_P10.16mm_Horizontal, F.Cu at (69.1, 77.2)
- added R2: 4.7k, Resistor_THT:R_Axial_DIN0207_L6.3mm_D2.5mm_P10.16mm_Horizontal, F.Cu at (82.5, 77.1)
- added R3: 4.7k, Resistor_THT:R_Axial_DIN0207_L6.3mm_D2.5mm_P10.16mm_Horizontal, F.Cu at (96.0, 77.1)
- moved BT1 45.4 mm to (44.5, 41.4)
- moved SW3 31.8 mm to (100.5, 83.6)
- moved SW2 28.5 mm to (87.0, 83.6)
- moved SW1 21.1 mm to (73.6, 83.7), turned to 90 degrees
- moved D7 2.55 mm to (118.2, 64.5)
- moved D8 2.55 mm to (112.2, 64.5)
- moved D1 2.55 mm to (94.2, 57.6)
- moved D10 2.55 mm to (100.2, 64.5)
- moved D11 2.55 mm to (94.2, 64.5)
- moved D2 2.55 mm to (100.2, 57.6)
- moved D3 2.55 mm to (106.2, 57.6)
- moved D4 2.55 mm to (112.2, 57.6)
- moved D5 2.55 mm to (118.2, 57.6)
- moved D6 2.55 mm to (124.2, 57.6)
- moved D9 2.55 mm to (106.2, 64.6)
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Routing:
- net Net-(U1-PD4): track 21.6 -> 53.9 mm
- net Net-(U1-PD3): track 17.6 -> 43.3 mm
- net +3.3V: track 90.5 -> 109.6 mm
- net MOSI: track 57.9 -> 41.6 mm
- net Net-(U1-PD2): track 18.4 -> 32.1 mm

Commit message: Add files via upload
Parts:
- removed R1, R2, R3: 4.7k, Resistor_THT:R_Axial_DIN0207_L6.3mm_D2.5mm_P10.16mm_Horizontal
- moved SW3 11.4 mm to (89.1, 83.3)
- moved SW2 7.71 mm to (79.2, 83.3)
- moved SW1 4.19 mm to (69.4, 83.3)
Connections:
- U1 pad 20: unconnected-(U1-AVCC-Pad20) -> +3.3V
Routing:
- net +3.3V: track 109.6 -> 80.0 mm
- net Net-(U1-PD4): track 53.9 -> 42.4 mm
- net Net-(U1-PD3): track 43.3 -> 35.5 mm
- net Net-(U1-PD2): track 32.1 -> 27.8 mm
- net MISO: track 31.8 -> 32.8 mm
- net SCK: track 42.3 -> 41.6 mm
Other:
- board text added: "lschneid(84352)"
