File: v5/kicad/binary_clock.kicad_sch (KiCad schematic)
At the start: 18 parts, among them J1 AVR-ISP-6, SW1 SW_Push, SW2 SW_Push, SW3 SW_Push, U1 ATmega48A-P, Y1 Crystal

Commit message: Add files via upload
Parts:
- BT1: footprint Battery:BatteryHolder_Keystone_104_1x23mm -> Battery:BatteryHolder_Keystone_103_1x20mm
- D1, D10, D11, D2, D3, D4, D5, D6, D7, D8, D9: footprint LED_SMD:LED_1210_3225Metric_Pad1.42x2.65mm_HandSolder -> LED_THT:LED_D3.0mm
- J1: footprint Connector_PinHeader_2.00mm:PinHeader_2x03_P2.00mm_Vertical -> Connector_PinSocket_2.54mm:PinSocket_2x03_P2.54mm_Vertical
- SW1, SW2, SW3: footprint Button_Switch_SMD:SW_Push_1P1T_NO_CK_KSC6xxJ -> Button_Switch_THT:SW_PUSH_6mm
- Y1: footprint Crystal:Crystal_AT310_D3.0mm_L10.0mm_Vertical -> Crystal:Crystal_DS10_D1.0mm_L4.3mm_Vertical
Connections:
- net +3.3V: no longer U1.20 (AVCC), U1.21 (AREF)
- net at D1.1 (K), D2.1 (K), D3.1 (K)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: no longer D10.1 (K), D11.1 (K), D7.1 (K), D8.1 (K), D9.1 (K)
- net at U1.16 (PB2): now also D10.1 (K), D11.1 (K), D7.1 (K), D8.1 (K), D9.1 (K)
- no-connect marks 2 -> 3

Commit message: Add files via upload
Parts:
- added R1, R2, R3: 4.7k, Resistor_THT:R_Axial_DIN0207_L6.3mm_D2.5mm_P10.16mm_Horizontal, symbol Device:R
Connections:
- net +3.3V: now also R1.2, R2.2, R3.2
- net at SW1.1, U1.4 (PD2): now also R1.1
- net at SW3.1, U1.6 (PD4): now also R3.1
- net at SW2.1, U1.5 (PD3): now also R2.1
Other:
- moved on the sheet: BT1, D1, D10, D11, D2, D3, D4, D5, D6, D7, D8, D9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

Commit message: Add files via upload
Parts:
- removed R1, R2, R3: 4.7k, Resistor_THT:R_Axial_DIN0207_L6.3mm_D2.5mm_P10.16mm_Horizontal, symbol Device:R
Connections:
- net +3.3V: now also U1.20 (AVCC)
- no-connect marks 3 -> 2
Other:
- moved on the sheet: SW1, SW2, SW3
